File: reader/reader.sch (KiCad schematic (older format))
At the start: 70 parts

Commit message: Schema work
Parts:
- removed C?: 100n, symbol Device:C_Small
- removed C?: 1u, symbol Device:C_Small
- removed U?: STM8L101F3P, Package_SO:TSSOP-20_4.4x6.5mm_P0.65mm, symbol MCU_ST_STM8:STM8L101F3P
- added C?: 100n, symbol Device:C_Small
- added C?: 1u, symbol Device:C_Small
- added R? (x8): 0, symbol Device:R_Small
- added U?: FC2004C03-NSWBBW-91*E, Display:NHD-0420H1Z, symbol Display_Character:NHD-0420H1Z
Connections:
- wire segments 136 -> 154
- no-connect marks 2 -> 3
Other:
- note added: "ssi_0 = 1, ssi_1 = 0\ni think, but lets be sure"
- note added: "vo is NC on my module"

Commit message: Schema done
Parts:
- removed D? (x16): 1N4001, symbol Device:D_Small
- removed SW?: a0, symbol Switch:SW_Push
- removed SW?: a1, symbol Switch:SW_Push
- removed SW?: a2, symbol Switch:SW_Push
- removed SW?: a3, symbol Switch:SW_Push
- removed SW?: b0, symbol Switch:SW_Push
- removed SW?: b1, symbol Switch:SW_Push
- removed SW?: b2, symbol Switch:SW_Push
- removed SW?: b3, symbol Switch:SW_Push
- removed SW?: c0, symbol Switch:SW_Push
- removed SW?: c1, symbol Switch:SW_Push
- removed SW?: c2, symbol Switch:SW_Push
- removed SW?: c3, symbol Switch:SW_Push
- removed SW?: d0, symbol Switch:SW_Push
- removed SW?: d1, symbol Switch:SW_Push
- removed SW?: d2, symbol Switch:SW_Push
- removed SW?: d3, symbol Switch:SW_Push
- removed Y?: 27.12MHz, symbol Device:Crystal_Small
- added C21, C28: 100n, Capacitor_SMD:C_0603_1608Metric_Pad1.05x0.95mm_HandSolder, symbol Device:C_Small
- added C23, C26: 33pF, Capacitor_SMD:C_0603_1608Metric_Pad1.05x0.95mm_HandSolder, symbol Device:C_Small
- added C27: 1u, Capacitor_SMD:C_0603_1608Metric_Pad1.05x0.95mm_HandSolder, symbol Device:C_Small
- added C29: 1u, good_things:NFM18PS105R0J3D, symbol Device:C_Feedthrough
- added FB4: 1k@100M, Inductor_SMD:L_0603_1608Metric_Pad1.05x0.95mm_HandSolder, symbol Device:Ferrite_Bead_Small
- added H1, H2, H3, H4: MountingHole_Pad, MountingHole:MountingHole_3.2mm_M3_DIN965_Pad, symbol Mechanical:MountingHole_Pad
- added J2: swd, Connector_PinHeader_2.54mm:PinHeader_1x03_P2.54mm_Vertical, symbol Connector_Generic:Conn_01x03
- added J3: Conn_01x06, Connector_PinHeader_2.54mm:PinHeader_1x06_P2.54mm_Vertical, symbol Connector_Generic:Conn_01x06
- added J4: v_sup, Connector_JST:JST_NV_B02P-NV_1x02_P5.00mm_Vertical, symbol Connector_Generic:Conn_01x02
- added R12, R13, R3: 10k, Resistor_SMD:R_0603_1608Metric_Pad1.05x0.95mm_HandSolder, symbol Device:R_Small
- added R14, R15: 0, Resistor_SMD:R_0603_1608Metric_Pad1.05x0.95mm_HandSolder, symbol Device:R_Small
- added R16, R17: 2k2, Resistor_SMD:R_0603_1608Metric_Pad1.05x0.95mm_HandSolder, symbol Device:R_Small
- added SW1: SW_Push, good_things:push_sw_purple, symbol Switch:SW_Push
- added U3: STM32G051GxU, Package_DFN_QFN:QFN-28_4x4mm_P0.5mm, symbol good_things:STM32G051GxU
- added Y1: 27.12MHz, Crystal:Crystal_SMD_2016-4Pin_2.0x1.6mm, symbol Device:Crystal_GND24
- added Y2: ABLS-24.000MHZ-20-B-3-H-T, Crystal:Crystal_SMD_HC49-SD, symbol Device:Crystal
- AE1: renamed from AE?; footprint (none) -> good_things:rfid_antenna
- C1, C10, C11, C12, C14, C15, C16, C17, C18, C2, C20, C22, C24, C25, C3, C4, C6, C7, C9: renamed from C?; footprint (none) -> Capacitor_SMD:C_0603_1608Metric_Pad1.05x0.95mm_HandSolder
- C13, C30: renamed from C?; footprint (none) -> Capacitor_SMD:C_0603_1608Metric_Pad1.05x0.95mm_HandSolder; farnell (none) -> 3013382
- C19: renamed from C?; footprint (none) -> good_things:NFM18PS105R0J3D
- C5, C8: renamed from C?; footprint (none) -> Capacitor_SMD:C_0603_1608Metric_Pad1.05x0.95mm_HandSolder; farnell (none) -> 3013453
- F1: renamed from F?; footprint (none) -> Fuse:Fuse_1210_3225Metric
- FB1, FB2, FB3: renamed from FB?; footprint (none) -> Inductor_SMD:L_0603_1608Metric_Pad1.05x0.95mm_HandSolder
- J1: renamed from J?; footprint (none) -> good_things:USB_MICRO_10118193-0001LF
- L1, L2: renamed from L?; footprint (none) -> Inductor_SMD:L_0603_1608Metric_Pad1.05x0.95mm_HandSolder; farnell (none) -> 2858966
- R1, R10, R11, R2, R4, R5, R6, R7, R8, R9: renamed from R?; footprint (none) -> Resistor_SMD:R_0603_1608Metric_Pad1.05x0.95mm_HandSolder
- U2: renamed from U?; footprint (none) -> Package_DFN_QFN:QFN-32-1EP_5x5mm_P0.5mm_EP3.65x3.65mm
- U4: renamed from U?; footprint Display:NHD-0420H1Z -> good_things:FC2004C03-NSWBBW-91
- gave numbers to parts that had none: 1
Connections:
- net labels added: encoder_a, encoder_b, i2c_scl, i2c_sda, lcd_d0, lcd_d1, lcd_d2, lcd_d3, lcd_d4, lcd_d5, lcd_d6, lcd_d7, lcd_e, lcd_rs, lcd_rw, nfc_irq_in, nfc_irq_out, nrst, spi_miso, spi_mosi, spi_nss, spi_sclk, swd_clk, swd_io, v_fused, vin, xtal_in, xtal_out
- net labels removed: matrix_0, matrix_1, matrix_2, matrix_3, matrix_a, matrix_b, matrix_c, matrix_d
- wire segments 154 -> 179
- no-connect marks 3 -> 4
Other:
- moved on the sheet: C14, C17, C30, F1, J1, U4

Commit message: Some placement and antenna
Parts:
- removed Y2: ABLS-24.000MHZ-20-B-3-H-T, Crystal:Crystal_SMD_HC49-SD, symbol Device:Crystal
- added Q1: CPH3350-TL-W, Package_TO_SOT_SMD:SOT-23_Handsoldering, symbol Device:Q_PMOS_GSD
- added R18: 10k, Resistor_SMD:R_0603_1608Metric_Pad1.05x0.95mm_HandSolder, symbol Device:R_Small
- added Y2: MCSJK-7U-27.00-12-10-60-B-10, Crystal:Crystal_SMD_Abracon_ABM8G-4Pin_3.2x2.5mm, symbol Device:Crystal_GND24_Small
- AE1: footprint good_things:rfid_antenna -> good_things:antenna_04p_04w_5turn
- C23, C26: value 33pF -> 16p
Connections:
- net labels added: 5v_filter, 5v_rf, i2c_scl_t, i2c_sda_t, mcu_vcc, mcu_vcc_t, v_potected
- wire segments 179 -> 192
- no-connect marks 4 -> 2
Other:
- moved on the sheet: C12, C17, C18, C21, C23, C26, C5, C8, F1, FB1, J1, J4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

Commit message: Pcb read done
Parts:
- removed H1, H2, H3, H4: MountingHole_Pad, MountingHole:MountingHole_3.2mm_M3_DIN965_Pad, symbol Mechanical:MountingHole_Pad
- removed J3: Conn_01x06, Connector_PinHeader_2.54mm:PinHeader_1x06_P2.54mm_Vertical, symbol Connector_Generic:Conn_01x06
- added J3: Conn_01x05, Connector_PinHeader_2.54mm:PinHeader_1x05_P2.54mm_Vertical, symbol Connector_Generic:Conn_01x05
- AE1: footprint good_things:antenna_04p_04w_5turn -> good_things:antenna_1m_07mm_3turn
Connections:
- net labels added: keypad_int, rfid_ss0, rfid_ss1, rfid_xin, rfid_xout, spi_clk_rfid, spi_miso_rfid, spi_mosi_rfid, spi_ss_rfid
- net labels removed: encoder_a, encoder_b
- wire segments 192 -> 203
- no-connect marks 2 -> 3
Other:
- moved on the sheet: AE1, C1, C10, C11, C13, C14, C15, C16, C17, C19, C2, C20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

Commit message: Touchups of main board
start design of keypad
see https://www.thevfdcollective.com/blog/stm32-and-sk6812-rgbw-led
Parts:
- removed C16, C22: 10n, Capacitor_SMD:C_0603_1608Metric_Pad1.05x0.95mm_HandSolder, symbol Device:C_Small
- removed C23, C26: 16p, Capacitor_SMD:C_0603_1608Metric_Pad1.05x0.95mm_HandSolder, symbol Device:C_Small
- removed FB2: 1k@200M, Inductor_SMD:L_0603_1608Metric_Pad1.05x0.95mm_HandSolder, symbol Device:Ferrite_Bead_Small
- removed J3: Conn_01x05, Connector_PinHeader_2.54mm:PinHeader_1x05_P2.54mm_Vertical, symbol Connector_Generic:Conn_01x05
- removed Y2: MCSJK-7U-27.00-12-10-60-B-10, Crystal:Crystal_SMD_Abracon_ABM8G-4Pin_3.2x2.5mm, symbol Device:Crystal_GND24_Small
- added J3: Conn_01x06, Connector_PinHeader_2.54mm:PinHeader_1x06_P2.54mm_Vertical, symbol Connector_Generic:Conn_01x06
- J1: symbol Connector:USB_B_Mini -> reader-rescue:USB_B_Mini-Connector
- U2: symbol good_things:ST25R95 -> reader-rescue:ST25R95-good_things
Connections:
- net +3V3: now also J3.1 (Pin_1)
- net +5V: now also FB3.2, J3.6 (Pin_6)
- net GND: now also J3.5 (Pin_5)
- net i2c_scl_t: now also J3.2 (Pin_2)
- net i2c_sda_t: now also J3.3 (Pin_3)
- net keypad_int: now also J3.4 (Pin_4)
- net xtal_in: no longer names the net of U3.1 (PC14)
- net xtal_out: no longer names the net of U3.2 (PC15)
- no-connect marks 3 -> 5
Other:
- moved on the sheet: C21, C9, R14, R15, R16, R17, R3, SW1

Commit message: Add keypad
Parts:
- added R19: 2k2, Resistor_SMD:R_0603_1608Metric_Pad1.05x0.95mm_HandSolder, symbol Device:R_Small
Connections:
- net +3V3: now also R19.1
- net keypad_int: now also R19.2
Other:
- moved on the sheet: R14, R15
Changed lines of the file:
@@
 	1    0    0    -1
 $EndComp
-Text GLabel 12500 2650 0    50   Input ~ 0
+Text GLabel 12050 2650 0    50   Input ~ 0
 i2c_sda
-Text GLabel 12500 2550 0    50   Input ~ 0
+Text GLabel 12050 2550 0    50   Input ~ 0
 i2c_scl
 $Comp
@@
 	1    0    0    -1
 $EndComp
-Connection ~ 13950 2650
-Connection ~ 13600 2550
 Wire Wire Line
 	13600 2150 13600 2550
@@
 	1    0    0    -1
 $EndComp
-Text GLabel 14200 2750 0    50   Input ~ 0
+Text GLabel 12050 2750 0    50   Input ~ 0
 keypad_int
 Wire Wire Line
 	13950 2150 13950 2650
-$Comp
-L Device:R_Small R14
-U 1 1 617FEA2B
-P 12700 2550
-F 0 "R14" V 12504 2550 50  0000 C CNN
-F 1 "0" V 12595 2550 50  0000 C CNN
-F 2 "Resistor_SMD:R_0603_1608Metric_Pad1.05x0.95mm_HandSolder" H 12700 2550 50  0001 C CNN
-F 3 "~" H 12700 2550 50  0001 C CNN
-	1    12700 2550
-	0    1    1    0
-$EndComp
-$Comp
-L Device:R_Small R15
-U 1 1 617FEC6C
-P 13050 2650
-F 0 "R15" V 12854 2650 50  0000 C CNN
-F 1 "0" V 12945 2650 50  0000 C CNN
-F 2 "Resistor_SMD:R_0603_1608Metric_Pad1.05x0.95mm_HandSolder" H 13050 2650 50  0001 C CNN
-F 3 "~" H 13050 2650 50  0001 C CNN
-	1    13050 2650
-	0    1    1    0
-$EndComp
-Wire Wire Line
-	13150 2650 13950 2650
-Wire Wire Line
-	12800 2550 13600 2550
-Wire Wire Line
-	12600 2550 12500 2550
-Wire Wire Line
-	12950 2650 12500 2650
 $Comp
 L Connector_Generic:Conn_01x02 J4
@@
 Text Label 5100 1350 0    50   ~ 0
 5v_filter
-Text Label 13200 2550 0    50   ~ 0
-i2c_scl_t
-Text Label 13200 2650 0    50   ~ 0
-i2c_sda_t
 Wire Wire Line
 	5250 4000 4900 4000
@@
 Wire Wire Line
 	9400 8000 9800 8000
-Wire Wire Line
-	10000 8250 10250 8250
 Connection ~ 10000 8250
 Wire Wire Line
 	10000 8200 10000 8250
-Wire Wire Line
-	10250 8250 10650 8250
-Connection ~ 10250 8250
 Connection ~ 9400 8250
 Wire Wire Line
@@
 	1    0    0    -1
 $EndComp
-Wire Wire Line
-	10250 8250 10250 8200
 Connection ~ 9400 8000
 $Comp
@@
 	13950 2650 14500 2650
 Wire Wire Line
-	14500 2750 14200 2750
-Wire Wire Line
 	7650 2900 8100 2900
 Wire Wire Line
@@
 	1    0    0    -1
 $EndComp
+Wire Wire Line
+	10000 8250 10650 8250
+Text Label 12800 2650 0    50   ~ 0
+i2c_sda_t
+Text Label 12800 2550 0    50   ~ 0
+i2c_scl_t
+Wire Wire Line
+	12500 2650 12050 2650
+Wire Wire Line
+	12150 2550 12050 2550
+$Comp
+L Device:R_Small R15
+U 1 1 617FEC6C
+P 12600 2650
+F 0 "R15" V 12404 2650 50  0000 C CNN
+F 1 "0" V 12495 2650 50  0000 C CNN
+F 2 "Resistor_SMD:R_0603_1608Metric_Pad1.05x0.95mm_HandSolder" H 12600 2650 50  0001 C CNN
+F 3 "~" H 12600 2650 50  0001 C CNN
+	1    12600 2650
+	0    1    1    0
+$EndComp
+$Comp
+L Device:R_Small R14
+U 1 1 617FEA2B
+P 12250 2550
+F 0 "R14" V 12054 2550 50  0000 C CNN
+F 1 "0" V 12145 2550 50  0000 C CNN
+F 2 "Resistor_SMD:R_0603_1608Metric_Pad1.05x0.95mm_HandSolder" H 12250 2550 50  0001 C CNN
+F 3 "~" H 12250 2550 50  0001 C CNN
+	1    12250 2550
+	0    1    1    0
+$EndComp
+Wire Wire Line
+	12050 2750 13250 2750
+Wire Wire Line
+	12700 2650 13950 2650
+Connection ~ 13950 2650
+Connection ~ 13600 2550
+$Comp
+L power:+3V3 #PWR0103
+U 1 1 616B91B8
+P 13250 1950
+F 0 "#PWR0103" H 13250 1800 50  0001 C CNN
+F 1 "+3V3" H 13265 2123 50  0000 C CNN
+F 2 "" H 13250 1950 50  0001 C CNN
+F 3 "" H 13250 1950 50  0001 C CNN
+	1    13250 1950
+	1    0    0    -1
+$EndComp
+$Comp
+L Device:R_Small R19
+U 1 1 616B91BE
+P 13250 2050
+F 0 "R19" H 13309 2096 50  0000 L CNN
+F 1 "2k2" H 13309 2005 50  0000 L CNN
+F 2 "Resistor_SMD:R_0603_1608Metric_Pad1.05x0.95mm_HandSolder" H 13250 2050 50  0001 C CNN
+F 3 "~" H 13250 2050 50  0001 C CNN
+	1    13250 2050
+	1    0    0    -1
+$EndComp
+Wire Wire Line
+	12350 2550 13600 2550
+Wire Wire Line
+	13250 2150 13250 2750
+Connection ~ 13250 2750
+Wire Wire Line
+	13250 2750 14500 2750
 $EndSCHEMATC

Commit message: fix footprint of inductor
Parts:
- L1, L2: footprint Inductor_SMD:L_0603_1608Metric_Pad1.05x0.95mm_HandSolder -> Inductor_SMD:L_0805_2012Metric
Changed lines of the file:
@@
 F 0 "L1" V 4319 2700 50  0000 C CNN
 F 1 "560n" V 4410 2700 50  0000 C CNN
-F 2 "Inductor_SMD:L_0603_1608Metric_Pad1.05x0.95mm_HandSolder" H 4500 2700 50  0001 C CNN
+F 2 "Inductor_SMD:L_0805_2012Metric" H 4500 2700 50  0001 C CNN
 F 3 "~" H 4500 2700 50  0001 C CNN
 F 4 "2858966" V 4500 2700 50  0001 C CNN "farnell"
@@
 F 0 "L2" V 4319 3550 50  0000 C CNN
 F 1 "560n" V 4410 3550 50  0000 C CNN
-F 2 "Inductor_SMD:L_0603_1608Metric_Pad1.05x0.95mm_HandSolder" H 4500 3550 50  0001 C CNN
+F 2 "Inductor_SMD:L_0805_2012Metric" H 4500 3550 50  0001 C CNN
 F 3 "~" H 4500 3550 50  0001 C CNN
 F 4 "2858966" V 4500 3550 50  0001 C CNN "farnell"
